File: bm1397.kicad_sch (KiCad schematic)
At the start: 58 parts, among them IC1 BM1397_mode1, J3 Conn_01x05, U2 LN1134A182MR-G, U3 SN74LVC1T45DBVR, U4 SGM2036-ADJYN5G/TR, U5 SN74LVC1T45DBVR, U8 SN74LVC1T45DBVR, X1 OT322525MJBA4SL

Commit message: added initial BOM
Parts:
- C20: DK (none) -> 478-KGM05AR51A225MHCT-ND; PARTNO (none) -> KGM05AR51A225MH
- R1, R2: PARTNO (none) -> RT0402BRE071KL
- R3, R4, R5: DK (none) -> RMCF0402ZT0R00; PARTNO (none) -> RMCF0402ZT0R00CT-ND
- TP1, TP10, TP11, TP12, TP13, TP14, TP17, TP19, TP23, TP24, TP32, TP5, TP6, TP7, TP8, TP9: now left out of the parts list
Changed lines of the file:
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@@
   )
   (symbol (lib_id "Connector:TestPoint") (at 37.465 82.55 90) (mirror x) (unit 1)
-    (in_bom yes) (on_board yes) (dnp no)
+    (in_bom no) (on_board yes) (dnp no)
     (property "Reference" "TP24" (at 31.115 82.55 90)
       (effects (font (size 1.27 1.27)))
@@
   )
   (symbol (lib_id "Connector:TestPoint") (at 207.645 94.615 90) (mirror x) (unit 1)
-    (in_bom yes) (on_board yes) (dnp no)
+    (in_bom no) (on_board yes) (dnp no)
     (property "Reference" "TP23" (at 201.295 94.615 90)
       (effects (font (size 1.27 1.27)))
@@
       (effects (font (size 1.27 1.27)) hide)
     )
-    (property "DK" "" (at 128.27 148.59 0)
-      (effects (font (size 1.778 1.5113)) (justify left bottom) hide)
-    )
-    (property "PARTNO" "" (at 128.27 148.59 0)
+    (property "DK" "478-KGM05AR51A225MHCT-ND" (at 128.27 148.59 0)
+      (effects (font (size 1.778 1.5113)) (justify left bottom) hide)
+    )
+    (property "PARTNO" "KGM05AR51A225MH" (at 128.27 148.59 0)
       (effects (font (size 1.27 1.27)) hide)
     )
@@
       (effects (font (size 1.27 1.27)) hide)
     )
+    (property "PARTNO" "RT0402BRE071KL" (at 52.705 90.805 0)
+      (effects (font (size 1.27 1.27)) hide)
+    )
     (pin "1")
     (pin "2")
@@
       (effects (font (size 1.27 1.27)) hide)
     )
+    (property "PARTNO" "RT0402BRE071KL" (at 40.64 88.9 0)
+      (effects (font (size 1.27 1.27)) hide)
+    )
     (pin "1")
     (pin "2")
@@
   )
   (symbol (lib_id "Connector:TestPoint") (at 128.27 74.93 270) (mirror x) (unit 1)
-    (in_bom yes) (on_board yes) (dnp no)
+    (in_bom no) (on_board yes) (dnp no)
     (property "Reference" "TP7" (at 134.62 74.93 90)
       (effects (font (size 1.27 1.27)))
@@
       (effects (font (size 1.27 1.27)) hide)
     )
-    (property "DK" "" (at 69.215 74.93 0)
-      (effects (font (size 1.27 1.27)) hide)
-    )
-    (property "PARTNO" "" (at 69.215 74.93 0)
+    (property "DK" "RMCF0402ZT0R00" (at 69.215 74.93 0)
+      (effects (font (size 1.27 1.27)) hide)
+    )
+    (property "PARTNO" "RMCF0402ZT0R00CT-ND" (at 69.215 74.93 0)
       (effects (font (size 1.27 1.27)) hide)
     )
@@
   )
   (symbol (lib_id "Connector:TestPoint") (at 140.335 80.01 270) (mirror x) (unit 1)
-    (in_bom yes) (on_board yes) (dnp no)
+    (in_bom no) (on_board yes) (dnp no)
     (property "Reference" "TP32" (at 146.685 80.01 90)
       (effects (font (size 1.27 1.27)))
@@
       (effects (font (size 1.27 1.27)) hide)
     )
-    (property "DK" "" (at 78.74 72.39 0)
-      (effects (font (size 1.27 1.27)) hide)
-    )
-    (property "PARTNO" "" (at 78.74 72.39 0)
+    (property "DK" "RMCF0402ZT0R00" (at 78.74 72.39 0)
+      (effects (font (size 1.27 1.27)) hide)
+    )
+    (property "PARTNO" "RMCF0402ZT0R00CT-ND" (at 78.74 72.39 0)
       (effects (font (size 1.27 1.27)) hide)
     )
@@
   )
   (symbol (lib_id "Connector:TestPoint") (at 207.645 45.085 90) (mirror x) (unit 1)
-    (in_bom yes) (on_board yes) (dnp no)
+    (in_bom no) (on_board yes) (dnp no)
     (property "Reference" "TP14" (at 201.295 45.085 90)
       (effects (font (size 1.27 1.27)))
@@
   )
   (symbol (lib_id "Connector:TestPoint") (at 128.27 72.39 270) (mirror x) (unit 1)
-    (in_bom yes) (on_board yes) (dnp no)
+    (in_bom no) (on_board yes) (dnp no)
     (property "Reference" "TP6" (at 134.62 72.39 90)
       (effects (font (size 1.27 1.27)))
@@
   )
   (symbol (lib_id "Connector:TestPoint") (at 128.27 82.55 270) (mirror x) (unit 1)
-    (in_bom yes) (on_board yes) (dnp no)
+    (in_bom no) (on_board yes) (dnp no)
     (property "Reference" "TP9" (at 134.62 82.55 90)
       (effects (font (size 1.27 1.27)))
@@
       (effects (font (size 1.27 1.27)) hide)
     )
-    (property "DK" "" (at 78.74 77.47 0)
-      (effects (font (size 1.27 1.27)) hide)
-    )
-    (property "PARTNO" "" (at 78.74 77.47 0)
+    (property "DK" "RMCF0402ZT0R00" (at 78.74 77.47 0)
+      (effects (font (size 1.27 1.27)) hide)
+    )
+    (property "PARTNO" "RMCF0402ZT0R00CT-ND" (at 78.74 77.47 0)
       (effects (font (size 1.27 1.27)) hide)
     )
@@
   )
   (symbol (lib_id "Connector:TestPoint") (at 207.645 69.85 90) (mirror x) (unit 1)
-    (in_bom yes) (on_board yes) (dnp no)
+    (in_bom no) (on_board yes) (dnp no)
     (property "Reference" "TP19" (at 201.295 69.85 90)
       (effects (font (size 1.27 1.27)))
@@
   )
   (symbol (lib_id "Connector:TestPoint") (at 135.255 168.275 270) (mirror x) (unit 1)
-    (in_bom yes) (on_board yes) (dnp no)
+    (in_bom no) (on_board yes) (dnp no)
     (property "Reference" "TP13" (at 141.605 168.275 90)
       (effects (font (size 1.27 1.27)))
@@
   )
   (symbol (lib_id "Connector:TestPoint") (at 128.27 80.01 270) (mirror x) (unit 1)
-    (in_bom yes) (on_board yes) (dnp no)
+    (in_bom no) (on_board yes) (dnp no)
     (property "Reference" "TP8" (at 134.62 80.01 90)
       (effects (font (size 1.27 1.27)))
@@
   )
   (symbol (lib_id "Connector:TestPoint") (at 36.83 161.29 90) (mirror x) (unit 1)
-    (in_bom yes) (on_board yes) (dnp no)
+    (in_bom no) (on_board yes) (dnp no)
     (property "Reference" "TP5" (at 30.48 161.29 90)
       (effects (font (size 1.27 1.27)))
@@
   )
   (symbol (lib_id "Connector:TestPoint") (at 145.415 88.265 270) (mirror x) (unit 1)
-    (in_bom yes) (on_board yes) (dnp no)
+    (in_bom no) (on_board yes) (dnp no)
     (property "Reference" "TP11" (at 151.765 88.265 90)
       (effects (font (size 1.27 1.27)))
@@
   )
   (symbol (lib_id "Connector:TestPoint") (at 146.05 94.615 270) (mirror x) (unit 1)
-    (in_bom yes) (on_board yes) (dnp no)
+    (in_bom no) (on_board yes) (dnp no)
     (property "Reference" "TP12" (at 152.4 94.615 90)
       (effects (font (size 1.27 1.27)))
@@
   )
   (symbol (lib_id "Connector:TestPoint") (at 128.27 95.25 270) (mirror x) (unit 1)
-    (in_bom yes) (on_board yes) (dnp no)
+    (in_bom no) (on_board yes) (dnp no)
     (property "Reference" "TP10" (at 134.62 95.25 90)
       (effects (font (size 1.27 1.27)))
@@
   )
   (symbol (lib_id "Connector:TestPoint") (at 141.605 142.24 270) (mirror x) (unit 1)
-    (in_bom yes) (on_board yes) (dnp no)
+    (in_bom no) (on_board yes) (dnp no)
     (property "Reference" "TP17" (at 147.955 142.24 90)
       (effects (font (size 1.27 1.27)))
@@
   )
   (symbol (lib_id "Connector:TestPoint") (at 55.88 113.03 0) (mirror x) (unit 1)
-    (in_bom yes) (on_board yes) (dnp no)
+    (in_bom no) (on_board yes) (dnp no)
     (property "Reference" "TP1" (at 55.88 119.38 90)
       (effects (font (size 1.27 1.27)))
